File: hw/sch_pcb/LION2CELL02.kicad_pcb (KiCad board)
At the start: 2 copper layers, 80.8 x 60.5 mm, 104 parts, among them J1 USBC_USB4105-GF-A, J10 HEADER_2x01_PARALLEL, J11 HEADER_1x02, J12 HEADER_2x05_PARALLEL, J2 CONN1_1, J3 CONN1_1, J4 JUMP_4X2, J5 HEADER_2x03_PARALLEL, J6 HEADER_2x01_PARALLEL, J7 HEADER_2x01_PARALLEL, J8 CONN1_1, J9 CONN1_1, Q1 DMTH3002LPS, Q2 AP2305AGN-HF-3, Q3 DMTH3002LPS, Q5 DMTH3002LPS, SW1 SW_Push, SW2 SW_Push, U1 BQ25792RQMR1, U2 LMR14050, U3 BQ40z50-R2

Commit message: Update USTids.
Parts:
- C2, C5: value 0.1u -> 100nF
- R19, R27, R28: value 5.1k -> 5k1
- TH1, TH2: value 10k -> NCP21XV103J03RA
