File: hw/sch_pcb/power_Input.kicad_sch (KiCad schematic)
At the start: 40 parts, among them J1 USBC_USB4105-GF-A, J6 HEADER_2x01_PARALLEL, J7 HEADER_2x01_PARALLEL, J8 CONN1_1, J9 CONN1_1, Q1 DMTH3002LPS, U1 BQ25792RQMR1

Commit message: Fix whitespaces around USTids.
Parts:
- C2, C29: UST_ID 5c70984712875079b91f8b4c -> 5c70984712875079b91f8b4c
- C20: value 4.7u -> 4u7; UST_ID (none) -> 5e3ff8fc1287502a33bad7a3
Changed lines of the file:
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@@
 		(dnp no)
 		(property "Reference" "C20"
-			(at 217.17 104.14 0)
+			(at 220.98 111.76 0)
 			(effects
 				(font
@@
 			)
 		)
-		(property "Value" "4.7u"
-			(at 218.44 106.68 0)
+		(property "Value" "4u7"
+			(at 220.98 109.22 0)
 			(effects
 				(font
@@
 			)
 		)
+		(property "UST_ID" "5e3ff8fc1287502a33bad7a3"
+			(at 219.71 110.49 0)
+			(effects
+				(font
+					(size 1.27 1.27)
+				)
+				(hide yes)
+			)
+		)
 		(pin "1"
 		)
@@
 			)
 		)
-		(property "UST_ID" " 5c70984712875079b91f8b4c"
+		(property "UST_ID" "5c70984712875079b91f8b4c"
 			(at 154.94 66.04 0)
 			(effects
@@
 			)
 		)
-		(property "UST_ID" " 5c70984712875079b91f8b4c "
+		(property "UST_ID" "5c70984712875079b91f8b4c"
 			(at 49.53 144.78 0)
 			(effects

Commit message: Fix components identification.
Parts:
- C1: MFPN C0805 1u -> (none); MPN C0805 1u -> (none); UST_ID 5c70984712875079b91f8b45 -> 5c70984712875079b91f8b4c
Changed lines of the file:
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@@
 			)
 		)
-		(property "MFPN" "C0805 1u"
+		(property "UST_ID" "5c70984712875079b91f8b4c"
 			(at 73.66 77.47 0)
 			(effects
-				(font
-					(size 1 1)
-				)
-				(hide yes)
-			)
-		)
-		(property "UST_ID" "5c70984712875079b91f8b45"
-			(at 73.66 77.47 0)
-			(effects
-				(font
-					(size 1 1)
-				)
-				(hide yes)
-			)
-		)
-		(property "MPN" "C0805 1u"
-			(at 73.66 77.47 0)
-			(effects
