File: hw/sch_pcb/power_output.kicad_sch (KiCad schematic)
At the start: 20 parts, among them J12 HEADER_2x05_PARALLEL, J2 CONN1_1, J3 CONN1_1, J4 JUMP_4X2, J5 HEADER_2x03_PARALLEL, U2 LMR14050

Commit message: Update USTids.
Parts:
- R13, R14, R15: UST_ID (none) -> 5c70984612875079b91f899f
Changed lines of the file:
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@@
 			)
 		)
-		(property "UST_ID" ""
+		(property "UST_ID" "5c70984612875079b91f899f"
 			(at 226.06 29.21 0)
 			(effects
@@
 			)
 		)
-		(property "UST_ID" ""
+		(property "UST_ID" "5c70984612875079b91f899f"
 			(at 232.41 29.21 0)
 			(effects
@@
 			)
 		)
-		(property "UST_ID" ""
+		(property "UST_ID" "5c70984612875079b91f899f"
 			(at 193.04 127 0)
 			(effects

Commit message: Fix components identification.
Parts:
- R12: value 15k8 -> 15k; UST_ID 6087b414128750769ee590a1 -> 5c70984712875079b91f8b6a
Changed lines of the file:
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@@
 			)
 		)
-		(property "Value" "15k8"
+		(property "Value" "15k"
 			(at 100.33 120.6499 0)
 			(effects
@@
 			)
 		)
-		(property "UST_ID" "6087b414128750769ee590a1"
+		(property "UST_ID" "5c70984712875079b91f8b6a"
 			(at 97.79 119.38 0)
 			(effects
